File: controller/controller.kicad_pcb (KiCad board)
At the start: 2 copper layers, 59.7 x 110.5 mm, 13 parts, among them IC1 TCST2103, J1 Screw_Terminal_01x08, U1 74HC590

Commit message: recent changes
Parts:
- removed ? (x6): , 
- removed IC1: TCST2103, TCST2103:TCST2103
- removed R1: 1000R, Resistor_THT:R_Axial_DIN0309_L9.0mm_D3.2mm_P12.70mm_Horizontal
- removed R2: 215R, Resistor_THT:R_Axial_DIN0309_L9.0mm_D3.2mm_P12.70mm_Horizontal
- removed U1: 74HC590, Package_DIP:DIP-16_W7.62mm_LongPads
- moved A2 435.4 mm to (603.2, 139.7)
- moved A1 424.0 mm to (578.8, 144.8), turned to 0 degrees
- moved J1 385.1 mm to (579.7, 133.0), turned to 0 degrees
Connections:
- A1 pad 11: Net-(A1-SCK/IO5) -> unconnected-(A1-SCK/IO5-Pad11)
- A1 pad 12: Net-(A1-MOSI/IO18) -> unconnected-(A1-MOSI/IO18-Pad12)
- A1 pad 13: Net-(A1-MISO/IO19) -> unconnected-(A1-MISO/IO19-Pad13)
- A1 pad 16: Net-(A1-IO21) -> unconnected-(A1-IO21-Pad16)
- A1 pad 22: Net-(A1-A9/IO33) -> unconnected-(A1-A9/IO33-Pad22)
- A1 pad 23: Net-(A1-A10/IO27) -> unconnected-(A1-A10/IO27-Pad23)
- A1 pad 24: Net-(A1-A11/IO12) -> unconnected-(A1-A11/IO12-Pad24)
- A1 pad 25: Net-(A1-A12/IO13) -> unconnected-(A1-A12/IO13-Pad25)
Routing:
- net Net-(U1-CPC): track 80.6 -> 0.00 mm
- net Net-(A1-IO21): track 71.1 -> 0.00 mm
- net Net-(A1-SCK/IO5): track 69.7 -> 0.00 mm
- net Net-(A1-MOSI/IO18): track 67.9 -> 0.00 mm
- net Net-(A1-MISO/IO19): track 66.1 -> 0.00 mm
- net Net-(IC1-PadT+): track 50.0 -> 0.00 mm
- net Net-(A1-A10/IO27): track 46.9 -> 0.00 mm
- net Net-(A1-A11/IO12): track 43.3 -> 0.00 mm
- net Net-(A1-A9/IO33): track 40.7 -> 0.00 mm
- net Net-(A1-A12/IO13): track 38.2 -> 0.00 mm
- net Net-(A1-A6/IO14): track 37.7 -> 0.00 mm
- net Net-(IC1-PadD+): track 31.9 -> 0.00 mm
- net Net-(A1-A7/IO32): track 30.8 -> 0.00 mm, vias 2 -> 0
- net Net-(A2-VMOT): track 27.7 -> 0.00 mm
- net +5V: track 26.2 -> 0.00 mm
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- removed copper zone on B.Cu, net GND
- removed copper zone on F.Cu, net GND
Other:
- board outline removed
